File: ram_rom_sio_cpu.sch (KiCad schematic (older format))
At the start: 20 parts, among them J4 Port A, U1 Z84C0010AEG, U2 Z84C4310AEG, U3 SST39LF040, U4 AS6C4008A-55ZIN

Commit message: gnd plane changes
Parts:
- U1: symbol SMC-80:Z84C0010AEG -> SMC-80_DE10-rescue:Z84C0010AEG-SMC-80
- U2: symbol SMC-80:Z84C4310AEG -> SMC-80_DE10-rescue:Z84C4310AEG-SMC-80
Changed lines of the file:
@@
 $EndComp
 $Comp
-L SMC-80:Z84C0010AEG U1
+L SMC-80_DE10-rescue:Z84C0010AEG-SMC-80 U1
 U 1 1 5F309FF5
 P 2900 2300
@@
 $EndComp
 $Comp
-L SMC-80:Z84C4310AEG U2
+L SMC-80_DE10-rescue:Z84C4310AEG-SMC-80 U2
 U 1 1 5DAA1781
 P 2900 5850
